File: Board files/sensor.brd (EAGLE design)
At the start: 25.4 x 59.7 mm, 34 parts, among them Q1 BCM847DS, U1 TL974, U2 TL974

Commit message: Fixed level shifter resistor values
Parts:
- R14: value 10K -> 68K
- R15: value 68K -> 10K
- R16: value 40.2K -> 10K
- R17: value 10K -> 2K
Changed lines of the file:
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@@
 <element name="R13" library="SparkFun-Resistors" package="0805" value="499K" x="7.62" y="25.4" rot="R90"/>
 <element name="C4" library="SparkFun-Capacitors" package="0805" value="0.1uF" x="3.81" y="25.4" rot="R90"/>
-<element name="R14" library="SparkFun-Resistors" package="0805" value="10K" x="3.81" y="20.32" rot="R90"/>
-<element name="R15" library="SparkFun-Resistors" package="0805" value="68K" x="7.62" y="10.16" rot="R90"/>
-<element name="R16" library="SparkFun-Resistors" package="0805" value="40.2K" x="15.24" y="10.16" rot="R270"/>
-<element name="R17" library="SparkFun-Resistors" package="0805" value="10K" x="11.43" y="10.16" rot="R90"/>
+<element name="R14" library="SparkFun-Resistors" package="0805" value="68K" x="3.81" y="20.32" rot="R90"/>
+<element name="R15" library="SparkFun-Resistors" package="0805" value="10K" x="7.62" y="10.16" rot="R90"/>
+<element name="R16" library="SparkFun-Resistors" package="0805" value="10K" x="15.24" y="10.16" rot="R270"/>
+<element name="R17" library="SparkFun-Resistors" package="0805" value="2K" x="11.43" y="10.16" rot="R90"/>
 <element name="C7" library="SparkFun-Capacitors" package="0805" value="0.1uF" x="19.05" y="19.685" rot="R90"/>
 <element name="C8" library="SparkFun-Capacitors" package="0805" value="0.1uF" x="19.05" y="15.875" rot="R90"/>
